Commit message: gripper added in Urdf

File: src/igus_rebel_description/urdf/igus_rebel.urdf (robot description, URDF)
Before this commit: robot igus_rebel, 9 links, 8 joints
Links:
- added link gripper, mass 0.1; collision mesh filename=package://igus_rebel_description/meshes/robolink_rebel/ZF-G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 scale=0.001 0.001 0.001; visual mesh filename=package://igus_rebel_description/meshes/robolink_rebel/ZF-G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 scale=0.001 0.001 0.001
Joints:
- added joint gripper_joint: type fixed, parent link_8, child gripper, origin xyz=0 -0.02 0 rpy=1.57 0 0

File: src/igus_rebel_description/urdf/igus_rebel2.urdf (robot description, URDF)
Before this commit: robot igus_rebel, 12 links, 11 joints
Links:
- added link gripper, mass 0.1; collision mesh filename=file://$(find igus_rebel_description)/meshes/robolink_rebel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 scale=0.001 0.001 0.001; visual mesh filename=file://$(find igus_rebel_description)/meshes/robolink_rebel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 scale=0.001 0.001 0.001
Joints:
- added joint gripper_joint: type fixed, parent link6, child gripper, origin xyz=0 -0.02 0.054 rpy=1.57 0 0
