Commit message: simulation with moveit

File: src/igus_rebel_description/urdf/igus_rebel.urdf (robot description, URDF)
Before this commit: robot igus_rebel, 10 links, 9 joints
Links:
- removed link gripper
Joints:
- removed joint gripper_joint

File: src/igus_rebel_description/urdf/igus_rebel2.control.xacro (robot description, xacro)
@@ -2,5 +2,4 @@
 <!-- igus_rebel.control.xacro -->
 <robot xmlns:xacro="http://www.ros.org/wiki/xacro">
-    <!--
     <xacro:macro name="igus_rebel_control" params="arm_id hardware_protocol">
         <xacro:macro name="joint_control" params="joint">
@@ -36,12 +35,13 @@
         </ros2_control>
         <xacro:if value="${hardware_protocol == 'gazebo'}">
-        -->
-        <gazebo>
-                <plugin filename="ign_ros2_control-system" name="ign_ros2_control::IgnitionROS2ControlPlugin">
-                <robot_param>igus_rebel_description</robot_param>
-                <robot_param_node>robot_state_publisher</robot_param_node>
-                <parameters>$(find rebel_ros2_controllers)/config/ros2_controllers.yaml</parameters>
-                <controller_manager_name>controller_manager</controller_manager_name>
-            </plugin>
-        </gazebo>
+            <gazebo>
+                <plugin filename="libgz_ros2_control-system.so" name="gz_ros2_control::GazeboSimROS2ControlPlugin">
+                    <robot_param>robot_description</robot_param>
+                    <robot_param_node>robot_state_publisher</robot_param_node>
+                    <parameters>$(find igus_rebel_moveit_config)/config/ros_controllers.yaml</parameters>
+                    <controller_manager_name>controller_manager</controller_manager_name>
+                </plugin>
+            </gazebo>
+        </xacro:if>
+    </xacro:macro>
 </robot>

File: src/igus_rebel_description/urdf/igus_rebel2.urdf (robot description, URDF)
Before this commit: robot igus_rebel, 12 links, 11 joints
Links:
- link base_link: geometry collision cylinder length=0.1 radius=0.09; visual mesh filename=file://$(find igus_rebel_description)/meshes/robolink_rebel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
- link link1: geometry collision box size=0.1 0.03 0.1; visual mesh filename=file://$(find igus_rebel_description)/meshes/robolink_rebel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
- link link2: geometry collision cylinder length=0.18 radius=0.06; visual mesh filename=file://$(find igus_rebel_description)/meshes/robolink_rebel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
- link link3: geometry collision box size=0.1 0.03 0.1; visual mesh filename=file://$(find igus_rebel_description)/meshes/robolink_rebel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
- link link4: geometry collision cylinder length=0.1 radius=0.05; visual mesh filename=file://$(find igus_rebel_description)/meshes/robolink_rebel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
- link link5: geometry collision box size=0.1 0.03 0.1; visual mesh filename=file://$(find igus_rebel_description)/meshes/robolink_rebel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
- link link6: geometry collision cylinder length=0.065 radius=0.04; visual mesh filename=file://$(find igus_rebel_description)/meshes/robolink_rebel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
- link motor1: geometry collision cylinder length=0.065 radius=0.05; visual mesh filename=file://$(find igus_rebel_description)/meshes/robolink_rebel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
- link motor2: geometry collision cylinder length=0.065 radius=0.05; visual mesh filename=file://$(find igus_rebel_description)/meshes/robolink_rebel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
- link motor3: geometry collision cylinder length=0.065 radius=0.05; visual mesh filename=file://$(find igus_rebel_description)/meshes/robolink_rebel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
- link motor4: geometry collision cylinder length=0.065 radius=0.05; visual mesh filename=file://$(find igus_rebel_description)/meshes/robolink_rebel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
- link motor5: geometry collision cylinder length=0.065 radius=0.04; visual mesh filename=file://$(find igus_rebel_description)/meshes/robolink_rebel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
Joints:
- joint joint1: axis 0 0 -1 -> 0 0 1

File: src/igus_rebel_description/urdf/igus_rebel_robot2.urdf.xacro (robot description, xacro)
@@ -2,10 +2,9 @@
 <robot xmlns:xacro="http://wiki.ros.org/xacro"
        name="igus_rebel" >
+  <xacro:arg name="hardware_protocol" default="rebel"/>
+  <!-- igus_rebel -->
   <xacro:include filename="$(find igus_rebel_description)/urdf/igus_rebel2.urdf" />
-  <xacro:include filename="$(find igus_rebel_description)/urdf/gazebo.xacro" />
-  <xacro:include filename="$(find rebel_ros2_controllers)/urdf/ros2_control.xacro"/>
-  <!--
-  <xacro:arg name="hardware_protocol" default="rebel"/>
-  <xacro:igus_rebel_control arm_id="rebel_arm" hardware_protocol="$(arg hardware_protocol)"/> -->
+  <xacro:include filename="$(find igus_rebel_description)/urdf/igus_rebel2.control.xacro"/>
+  <xacro:igus_rebel_control arm_id="rebel_arm" hardware_protocol="$(arg hardware_protocol)"/>
   <link name="world" />
   <joint name="world_joint" type="fixed">
