Commit message: ros2 controllers added

File: src/igus_rebel_description/urdf/igus_rebel2.control.xacro (robot description, xacro)
@@ -2,4 +2,5 @@
 <!-- igus_rebel.control.xacro -->
 <robot xmlns:xacro="http://www.ros.org/wiki/xacro">
+    <!--
     <xacro:macro name="igus_rebel_control" params="arm_id hardware_protocol">
         <xacro:macro name="joint_control" params="joint">
@@ -35,13 +36,12 @@
         </ros2_control>
         <xacro:if value="${hardware_protocol == 'gazebo'}">
-            <gazebo>
-                <plugin filename="libgz_ros2_control-system.so" name="gz_ros2_control::GazeboSimROS2ControlPlugin">
-                    <robot_param>robot_description</robot_param>
-                    <robot_param_node>robot_state_publisher</robot_param_node>
-                    <parameters>$(find igus_rebel_moveit_config)/config/ros_controllers.yaml</parameters>
-                    <controller_manager_name>controller_manager</controller_manager_name>
-                </plugin>
-            </gazebo>
-        </xacro:if>
-    </xacro:macro>
+        -->
+        <gazebo>
+                <plugin filename="ign_ros2_control-system" name="ign_ros2_control::IgnitionROS2ControlPlugin">
+                <robot_param>igus_rebel_description</robot_param>
+                <robot_param_node>robot_state_publisher</robot_param_node>
+                <parameters>$(find rebel_ros2_controllers)/config/ros2_controllers.yaml</parameters>
+                <controller_manager_name>controller_manager</controller_manager_name>
+            </plugin>
+        </gazebo>
 </robot>

File: src/igus_rebel_description/urdf/igus_rebel2.urdf (robot description, URDF)
Before this commit: robot igus_rebel, 13 links, 12 joints
Links:
- removed link gripper
Joints:
- removed joint gripper_joint

File: src/igus_rebel_description/urdf/igus_rebel_robot2.urdf.xacro (robot description, xacro)
@@ -2,9 +2,10 @@
 <robot xmlns:xacro="http://wiki.ros.org/xacro"
        name="igus_rebel" >
+  <xacro:include filename="$(find igus_rebel_description)/urdf/igus_rebel2.urdf" />
+  <xacro:include filename="$(find igus_rebel_description)/urdf/gazebo.xacro" />
+  <xacro:include filename="$(find rebel_ros2_controllers)/urdf/ros2_control.xacro"/>
+  <!--
   <xacro:arg name="hardware_protocol" default="rebel"/>
-  <!-- igus_rebel -->
-  <xacro:include filename="$(find igus_rebel_description)/urdf/igus_rebel2.urdf" />
-  <xacro:include filename="$(find igus_rebel_description)/urdf/igus_rebel2.control.xacro"/>
-  <xacro:igus_rebel_control arm_id="rebel_arm" hardware_protocol="$(arg hardware_protocol)"/>
+  <xacro:igus_rebel_control arm_id="rebel_arm" hardware_protocol="$(arg hardware_protocol)"/> -->
   <link name="world" />
   <joint name="world_joint" type="fixed">
