Commit message: camera monting and hsv

File: src/igus_rebel_description/urdf/igus_rebel2.urdf (robot description, URDF)
Before this commit: robot igus_rebel, 12 links, 11 joints
Links:
- added link gripper_base, mass 1.0; collision mesh filename=file://$(find igus_rebel_description)/meshes/gripper/grippe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 scale=0.001 0.001 0.001; visual mesh filename=file://$(find igus_rebel_description)/meshes/gripper/grippe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 scale=0.001 0.001 0.001
- added link gripper_left, mass 0.2; collision mesh filename=file://$(find igus_rebel_description)/meshes/gripper/left_l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 scale=0.001 0.001 0.001; visual mesh filename=file://$(find igus_rebel_description)/meshes/gripper/left_l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 scale=0.001 0.001 0.001
- added link gripper_right, mass 0.2; collision mesh filename=file://$(find igus_rebel_description)/meshes/gripper/right_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 scale=0.001 0.001 0.001; visual mesh filename=file://$(find igus_rebel_description)/meshes/gripper/right_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 scale=0.001 0.001 0.001
Joints:
- added joint gripper_left_joint: type fixed, parent gripper_base, child gripper_left, origin xyz=0 0 0 rpy=0 0 0, axis 0 0 1, limit lower=-1.57 upper=1.57 effort=10 velocity=1.0
- added joint gripper_mount_joint: type fixed, parent link6, child gripper_base, origin xyz=0 -0.02 0.054 rpy=1.570796 0 0
- added joint gripper_right_joint: type fixed, parent gripper_base, child gripper_right, origin xyz=0 0 0 rpy=0 0 0, axis 0 0 1, limit lower=-1.57 upper=1.57 effort=10 velocity=1.0

Commit message: aruco marker calib

File: src/igus_rebel_description/urdf/igus_rebel2.urdf (robot description, URDF)
Before this commit: robot igus_rebel, 15 links, 14 joints
Links:
- added link camera_link, mass 1.0; collision box size=0.12 0.12 0.07; visual box size=0.10 0.10 0.05
- added link camera_stand_horizontal, mass 1.0; collision box size=0.91 0.08 0.08; visual box size=0.87 0.05 0.05
- added link camera_stand_pole, mass 1.0; collision box size=0.08 0.08 0.78; visual box size=0.05 0.05 0.745
Joints:
- added joint camera_stand_to_camera: type fixed, parent camera_stand_horizontal, child camera_link, origin xyz=-0.395 0 -0.060 rpy=0 0 0
- added joint camera_stand_to_horizontal: type fixed, parent camera_stand_pole, child camera_stand_horizontal, origin xyz=0 0.435 0.3975 rpy=0 0 -1.5708
- added joint world_to_camera_stand: type fixed, parent world, child camera_stand_pole, origin xyz=0 -0.70 0.3725 rpy=0 0 0

Commit message: calibration files and recent files

File: src/igus_rebel_description/urdf/igus_rebel2.urdf (robot description, URDF)
Before this commit: robot igus_rebel, 18 links, 17 joints
Links:
- removed link camera_link
- added link camera_visual_link, mass 1.0; collision box size=0.12 0.12 0.07; visual box size=0.10 0.10 0.05
Joints:
- joint camera_stand_to_camera: child camera_link -> camera_visual_link
- joint world_to_camera_stand: origin xyz=0 -0.70 0.3725 rpy=0 0 0 -> xyz=0.31 -0.65 0.3725 rpy=0 0 0

Commit message: YOLO detection simulation

File: src/igus_rebel_description/urdf/igus_rebel2.urdf (robot description, URDF)
Before this commit: robot igus_rebel, 18 links, 17 joints
Links:
- removed link gripper_base
- removed link gripper_left
- removed link gripper_right
Joints:
- removed joint gripper_left_joint
- removed joint gripper_mount_joint
- removed joint gripper_right_joint
- joint world_to_camera_stand: origin xyz=0.31 -0.65 0.3725 rpy=0 0 0 -> xyz=0.31 -0.80 0.3725 rpy=0 0 0

File: src/igus_rebel_description/urdf/igus_rebel_robot2.urdf.xacro (robot description, xacro)
@@ -3,6 +3,15 @@
        name="igus_rebel" >
   <xacro:arg name="hardware_protocol" default="rebel"/>
-  <!-- igus_rebel -->
+  <xacro:property name="hw_protocol" value="$(arg hardware_protocol)"/>
+  <!-- igus_rebel arm and camera stand (no gripper in this file any more) -->
   <xacro:include filename="$(find igus_rebel_description)/urdf/igus_rebel2.urdf" />
+  <!-- Gripper, simulated moving fingers in Gazebo, real gripper meshes for everything else -->
+  <xacro:if value="${hw_protocol == 'gazebo'}">
+    <xacro:include filename="$(find igus_rebel_description)/urdf/sim_gripper.xacro"/>
+    <xacro:include filename="$(find igus_rebel_description)/urdf/sim_camera.xacro"/>
+  </xacro:if>
+  <xacro:unless value="${hw_protocol == 'gazebo'}">
+    <xacro:include filename="$(find igus_rebel_description)/urdf/gripper_real.xacro"/>
+  </xacro:unless>
   <xacro:include filename="$(find igus_rebel_description)/urdf/igus_rebel2.control.xacro"/>
   <xacro:igus_rebel_control arm_id="rebel_arm" hardware_protocol="$(arg hardware_protocol)"/>
